File: hardware/arpie_synch_module.sch (EAGLE design)
At the start: 44 parts, among them IC1 4584N

Commit message: rev3
Parts:
- removed INPUT, OUTPUT: STEREOJACK, adafruit:STEREOJACK
- added U$1, U$2: TRUCONNECTJACK, jason_eagle6:TRUCONNECTJACK
- R1: value 1M -> 10K
- R3: value 10K -> 1M
Connections:
- net +5V: no longer VCC.1, VCC1.1, VCC2.1
- net GND: now also R3.2, U$1.SLEEVE, U$2.SLEEVE; no longer GND.1, GND1.1, GND2.1, GND3.1, GND4.1, GND5.1, GND6.1, INPUT.1, OUTPUT.1, R1.2
- net N$11: now also R3.1, U$1.RING; no longer INPUT.5, R1.1
- net N$3: now also U$1.TIP, U$2.TIP, U$2.TIP_NC; no longer INPUT.2, OUTPUT.2, OUTPUT.3
- net N$4: now also R1.2, U$1.TIP_NC; no longer INPUT.3, R3.2
- net N$5: now also R1.1; no longer R3.1
- net N$9: now also U$1.RING_NC; no longer INPUT.4
Other:
- moved on the sheet: C1, R1, R2, R3
