File: hardware/arpie_synch_module.sch (EAGLE design)
At the start: 44 parts, among them IC1 4584N

Commit message: rev4
fix connection issue, add recess for socket barrel
Connections:
- net +5V: now also VCC.1
- net GND: now also GND.1
Changed lines of the file:
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@@
 <?xml version="1.0" encoding="utf-8"?>
 <!DOCTYPE eagle SYSTEM "eagle.dtd">
-<eagle version="6.4">
+<eagle version="6.6.0">
 <drawing>
 <settings>
@@
 <part name="U$1" library="jason_eagle6" deviceset="TRUCONNECTJACK" device=""/>
 <part name="U$2" library="jason_eagle6" deviceset="TRUCONNECTJACK" device=""/>
+<part name="SUPPLY4" library="supply2" deviceset="+5V" device=""/>
+<part name="GND13" library="SparkFun" deviceset="GND" device=""/>
 </parts>
 <sheets>
@@
 <instance part="U$1" gate="G$1" x="231.14" y="40.64"/>
 <instance part="U$2" gate="G$1" x="231.14" y="15.24"/>
+<instance part="SUPPLY4" gate="+5V" x="111.76" y="119.38"/>
+<instance part="GND13" gate="1" x="144.78" y="93.98"/>
 </instances>
 <busses>
@@
 <pinref part="U$1" gate="G$1" pin="SLEEVE"/>
 <wire x1="205.74" y1="45.72" x2="210.82" y2="45.72" width="0.1524" layer="91"/>
+<junction x="210.82" y="45.72"/>
 </segment>
 <segment>
@@
 <pinref part="U$2" gate="G$1" pin="SLEEVE"/>
 <wire x1="205.74" y1="20.32" x2="210.82" y2="20.32" width="0.1524" layer="91"/>
+<junction x="210.82" y="20.32"/>
 </segment>
 <segment>
@@
 <wire x1="152.4" y1="-5.08" x2="152.4" y2="-2.54" width="0.1524" layer="91"/>
 <junction x="152.4" y="-2.54"/>
+</segment>
+<segment>
+<pinref part="GND" gate="G$1" pin="1"/>
+<wire x1="152.4" y1="104.14" x2="144.78" y2="104.14" width="0.1524" layer="91"/>
+<wire x1="144.78" y1="104.14" x2="144.78" y2="96.52" width="0.1524" layer="91"/>
+<pinref part="GND13" gate="1" pin="GND"/>
 </segment>
 </net>
@@
 <pinref part="U$2" gate="G$1" pin="TIP_NC"/>
 <wire x1="205.74" y1="27.94" x2="210.82" y2="27.94" width="0.1524" layer="91"/>
+<junction x="210.82" y="55.88"/>
+<junction x="210.82" y="30.48"/>
+<junction x="210.82" y="27.94"/>
 </segment>
 </net>
@@
 <pinref part="U$1" gate="G$1" pin="TIP_NC"/>
 <wire x1="205.74" y1="53.34" x2="210.82" y2="53.34" width="0.1524" layer="91"/>
+<junction x="210.82" y="53.34"/>
 </segment>
 </net>
@@
 <pinref part="U$1" gate="G$1" pin="RING_NC"/>
 <wire x1="205.74" y1="48.26" x2="210.82" y2="48.26" width="0.1524" layer="91"/>
+<junction x="210.82" y="48.26"/>
+<junction x="157.48" y="60.96"/>
 </segment>
 </net>
@@
 <pinref part="U$1" gate="G$1" pin="RING"/>
 <wire x1="205.74" y1="50.8" x2="210.82" y2="50.8" width="0.1524" layer="91"/>
+<junction x="210.82" y="50.8"/>
 </segment>
 </net>
@@
 <junction x="139.7" y="5.08"/>
 </segment>
-</net>
+<segment>
+<pinref part="VCC" gate="G$1" pin="1"/>
+<wire x1="134.62" y1="111.76" x2="111.76" y2="111.76" width="0.1524" layer="91"/>
+<wire x1="111.76" y1="111.76" x2="111.76" y2="116.84" width="0.1524" layer="91"/>
+<pinref part="SUPPLY4" gate="+5V" pin="+5V"/>
+</segment>
+</net>
