File: hardware/arpie_synch_module.brd (EAGLE design)
At the start: 36.1 x 50.8 mm, 44 parts, among them IC1 4584N

Commit message: rev3
Parts:
- removed INPUT, OUTPUT: STEREOJACK, adafruit:STX3100
- added U$1, U$2: TRUCONNECTJACK, jason_eagle6:TRUCONNECTJACK
- R1: value 1M -> 10K
- R3: value 10K -> 1M
- moved R4 12.7 mm to (78.7, 30.5)
- moved R5 12.7 mm to (78.7, 27.9)
- moved R1 12.7 mm to (78.7, 38.1), turned to 0 degrees
- moved R2 12.7 mm to (78.7, 35.6)
- moved R3 12.7 mm to (78.7, 33.0), turned to 180 degrees
- moved C2 10.3 mm to (67.3, 33.0), turned to 180 degrees
- moved C1 2.58 mm to (78.7, 41.2), turned to 180 degrees
Connections:
- net +5V: no longer VCC.1, VCC1.1, VCC2.1
- net GND: now also R3.2, U$1.SLEEVE, U$2.SLEEVE; no longer GND.1, GND1.1, GND2.1, GND3.1, GND4.1, GND5.1, GND6.1, INPUT.1, OUTPUT.1, R1.2
- net N$11: now also R3.1, U$1.RING; no longer INPUT.5, R1.1
- net N$3: now also U$1.TIP, U$2.TIP, U$2.TIP_NC; no longer INPUT.2, OUTPUT.2, OUTPUT.3
- net N$4: now also R1.2, U$1.TIP_NC; no longer INPUT.3, R3.2
- net N$5: now also R1.1; no longer R3.1
- net N$9: now also U$1.RING_NC; no longer INPUT.4
Routing:
- net +5V: track 111.4 -> 72.6 mm, vias 1 -> 0
- net N$11: track 21.4 -> 8.67 mm
- net N$15: track 12.3 -> 4.34 mm
- net N$9: track 12.4 -> 6.13 mm
- net N$5: track 23.6 -> 29.8 mm
- net N$12: track 28.6 -> 24.4 mm
- net N$3: track 27.0 -> 25.0 mm
- net N$4: track 13.0 -> 13.8 mm
- net GND: track 0.76 -> 0.00 mm
Other:
- board size 36.1 x 50.8 mm -> 35.9 x 50.8 mm
- board text added: "rev 3"
- board text removed: "rev 2"

Commit message: rev4
fix connection issue, add recess for socket barrel
Connections:
- net +5V: now also VCC.1
- net GND: now also GND.1
Routing:
- net +5V: track 72.6 -> 75.9 mm
Other:
- outline, holes or cut-outs redrawn
- board text added: "rev 4"
- board text removed: "rev 3"
Changed lines of the file:
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@@
 <?xml version="1.0" encoding="utf-8"?>
 <!DOCTYPE eagle SYSTEM "eagle.dtd">
-<eagle version="6.4">
+<eagle version="6.6.0">
 <drawing>
 <settings>
@@
 <setting verticaltext="up"/>
 </settings>
-<grid distance="2" unitdist="mil" unit="mil" style="lines" multiple="1" display="yes" altdistance="0.001" altunitdist="inch" altunit="inch"/>
+<grid distance="0.05" unitdist="inch" unit="inch" style="lines" multiple="1" display="yes" altdistance="0.001" altunitdist="inch" altunit="inch"/>
 <layers>
 <layer number="1" name="Top" color="4" fill="1" visible="yes" active="yes"/>
@@
 <wire x1="60.6044" y1="46.7106" x2="62.2427" y2="48.265" width="0.4064" layer="20" curve="-90.010794"/>
 <wire x1="96.5149" y1="45.7022" x2="93.9064" y2="48.26" width="0.4064" layer="20" curve="81.267246"/>
-<wire x1="96.52" y1="10.16" x2="96.52" y2="45.72" width="0.4064" layer="20"/>
+<wire x1="96.52" y1="10.16" x2="96.52" y2="24.13" width="0.4064" layer="20"/>
+<wire x1="96.52" y1="31.75" x2="96.52" y2="36.83" width="0.4064" layer="20"/>
+<wire x1="96.52" y1="44.45" x2="96.52" y2="45.72" width="0.4064" layer="20"/>
 <wire x1="93.9064" y1="48.26" x2="62.23" y2="48.26" width="0.4064" layer="20"/>
 <text x="86.233" y="14.351" size="2.032" layer="21" font="vector" rot="R90">INT</text>
@@
 <text x="81.28" y="43.307" size="2.54" layer="22" font="vector" rot="MR270">IN</text>
 <text x="81.28" y="31.75" size="2.54" layer="22" font="vector" rot="MR270">OUT</text>
-<text x="63.246" y="46.228" size="1.778" layer="22" font="vector" rot="MR270">rev 3</text>
+<text x="63.246" y="46.228" size="1.778" layer="22" font="vector" rot="MR270">rev 4</text>
 <text x="84.709" y="5.588" size="1.778" layer="22" font="vector" rot="MR90">hotchk155</text>
 <rectangle x1="69.7738" y1="37.5666" x2="73.6854" y2="37.6174" layer="51"/>
@@
 <wire x1="80.3148" y1="43.942" x2="80.4164" y2="43.8404" width="0.3048" layer="51"/>
 <wire x1="80.4418" y1="44.4246" x2="80.4418" y2="43.815" width="0.3048" layer="51"/>
+<wire x1="96.52" y1="44.45" x2="95.25" y2="44.45" width="0.3048" layer="20"/>
+<wire x1="95.25" y1="44.45" x2="95.25" y2="36.83" width="0.3048" layer="20"/>
+<wire x1="95.25" y1="36.83" x2="96.52" y2="36.83" width="0.3048" layer="20"/>
+<wire x1="96.52" y1="31.75" x2="95.25" y2="31.75" width="0.3048" layer="20"/>
+<wire x1="95.25" y1="31.75" x2="95.25" y2="24.13" width="0.3048" layer="20"/>
+<wire x1="95.25" y1="24.13" x2="96.52" y2="24.13" width="0.3048" layer="20"/>
 </plain>
 <attributes>
@@
 <contactref element="U$1" pad="SLEEVE"/>
 <contactref element="U$2" pad="SLEEVE"/>
+<contactref element="GND" pad="1"/>
 </signal>
 <signal name="N$3">
@@
 <contactref element="C3" pad="+"/>
 <contactref element="C2" pad="1"/>
-<wire x1="61.722" y1="11.176" x2="61.722" y2="30.0482" width="0.6096" layer="16"/>
+<wire x1="61.722" y1="9.8044" x2="61.722" y2="30.0482" width="0.6096" layer="16"/>
 <wire x1="71.12" y1="29.21" x2="67.31" y2="29.21" width="0.6096" layer="16"/>
-<wire x1="67.31" y1="29.21" x2="66.04" y2="30.48" width="0.6096" layer="16"/>
+<wire x1="67.31" y1="29.21" x2="65.3796" y2="31.1404" width="0.6096" layer="16"/>
 <wire x1="71.12" y1="29.21" x2="71.12" y2="33.02" width="0.6096" layer="16"/>
 <wire x1="71.12" y1="33.02" x2="73.66" y2="35.56" width="0.6096" layer="16"/>
 <wire x1="73.66" y1="35.56" x2="74.93" y2="35.56" width="0.6096" layer="16"/>
-<wire x1="90.043" y1="6.35" x2="89.154" y2="5.461" width="0.6096" layer="16"/>
-<wire x1="89.154" y1="5.461" x2="69.723" y2="5.461" width="0.6096" layer="16"/>
+<wire x1="89.281" y1="5.461" x2="69.723" y2="5.461" width="0.6096" layer="16"/>
 <wire x1="69.723" y1="5.461" x2="67.31" y2="7.874" width="0.6096" layer="16"/>
 <wire x1="67.31" y1="7.874" x2="63.6524" y2="7.874" width="0.6096" layer="16"/>
 <wire x1="63.6524" y1="7.874" x2="61.722" y2="9.8044" width="0.6096" layer="16"/>
-<wire x1="61.722" y1="9.8044" x2="61.722" y2="11.176" width="0.6096" layer="16"/>
-<wire x1="66.04" y1="30.48" x2="65.3796" y2="31.1404" width="0.6096" layer="16"/>
 <wire x1="65.3796" y1="31.1404" x2="62.8142" y2="31.1404" width="0.6096" layer="16"/>
 <wire x1="62.8142" y1="31.1404" x2="61.722" y2="30.0482" width="0.6096" layer="16"/>
 <wire x1="68.5546" y1="33.02" x2="71.12" y2="33.02" width="0.6096" layer="16"/>
+<contactref element="VCC" pad="1"/>
+<wire x1="93.345" y1="6.35" x2="90.17" y2="6.35" width="0.6096" layer="16"/>
+<wire x1="90.17" y1="6.35" x2="89.281" y2="5.461" width="0.6096" layer="16"/>
 </signal>
 <signal name="N$14">
